Commit message: URDF edit

File: src/dm/robot_model/urdf/robot_model.urdf (robot description, URDF)
Before this commit: robot urdf_omnidirectional_manipulator, 11 links, 10 joints
Links:
- link Link_1: geometry collision mesh filename=package://robot_model/meshes/Link_1.STL; visual mesh filename=package://robot_model/meshes/Link_1.STL
- link Link_2: geometry collision mesh filename=package://robot_model/meshes/Link_2.STL; visual mesh filename=package://robot_model/meshes/Link_2.STL
- link Link_3: geometry collision mesh filename=package://robot_model/meshes/Link_3.STL; visual mesh filename=package://robot_model/meshes/Link_3.STL
- link Link_4: geometry collision mesh filename=package://robot_model/meshes/Link_4.STL; visual mesh filename=package://robot_model/meshes/Link_4.STL
- link Link_5: geometry collision mesh filename=package://robot_model/meshes/Link_5.STL; visual mesh filename=package://robot_model/meshes/Link_5.STL
- link base_link: geometry collision mesh filename=package://robot_model/meshes/base_link.STL; visual mesh filename=package://robot_model/meshes/base_link.STL
- link end_effector: geometry collision mesh filename=package://robot_model/meshes/end_effector.STL; visual mesh filename=package://robot_model/meshes/end_effector.STL
- link fl_wheel_link: geometry collision mesh filename=package://robot_model/meshes/fl_wheel_link.STL; visual mesh filename=package://robot_model/meshes/fl_wheel_link.STL
- link fr_wheel_link: geometry collision mesh filename=package://robot_model/meshes/fr_wheel_link.STL; visual mesh filename=package://robot_model/meshes/fr_wheel_link.STL
- link rl_wheel_link: geometry collision mesh filename=package://robot_model/meshes/rl_wheel_link.STL; visual mesh filename=package://robot_model/meshes/rl_wheel_link.STL
- link rr_wheel_link: geometry collision mesh filename=package://robot_model/meshes/rr_wheel_link.STL; visual mesh filename=package://robot_model/meshes/rr_wheel_link.STL
