File: pcb/wheels-pcb/wheels-pcb.kicad_pcb (KiCad board)
At the start: 2 copper layers, 16 parts, among them J1 Motor_1, J2 Motor_2, J3 Motor_3, J4 Motor_4, J5 Conn_01x03, U1 L293D, U2 L293D, U3 ESP32S_38P

Commit message: pcb-modification
Parts:
- J1, J2, J3, J4: footprint Connectors_JST:JST_EH_B06B-EH-A_06x2.50mm_Straight -> Connector_JST:JST_EH_B6B-EH-A_1x06_P2.50mm_Vertical
- J5: footprint Connectors_JST:JST_EH_S03B-EH_03x2.50mm_Angled -> Connector_JST:JST_EH_S3B-EH_1x03_P2.50mm_Horizontal
- moved D7 31.8 mm to (175.5, 105.3), turned to 90 degrees
- moved D6 27.7 mm to (175.5, 66.1), turned to -90 degrees
- moved J1 26.8 mm to (128.5, 61.7), turned to 180 degrees
- moved J4 25.0 mm to (175.5, 111.5)
- moved D3 24.6 mm to (128.5, 104.3), turned to 90 degrees
- moved D2 20.1 mm to (128.5, 66.6), turned to -90 degrees
- moved U1 20.0 mm to (113.5, 88.7), turned to 90 degrees
- moved U2 17.9 mm to (190.5, 81.1), turned to -90 degrees
- moved D8 17.5 mm to (187.9, 105.3), turned to 90 degrees
- moved J2 13.3 mm to (116.0, 111.2)
- moved D5 13.2 mm to (188.0, 66.2), turned to -90 degrees
- moved D4 12.6 mm to (116.0, 104.3), turned to 90 degrees
- moved J5 11.5 mm to (184.5, 121.7), turned to 180 degrees
- moved J3 11.5 mm to (188.0, 61.7), turned to 180 degrees
- moved U3 8.98 mm to (152.0, 54.5)
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Connections:
- U2 pad 9: unconnected-(U2-EN3,4-Pad9) -> Net-(U2-EN3,4)
- U3 pad 27: unconnected-(U3-GPIO16-Pad27) -> Net-(U2-EN3,4)
Routing:
- net GND: track 0.00 -> 338.0 mm
- net +5V: track 0.00 -> 222.3 mm
- net +12V: track 0.00 -> 153.9 mm
- net Net-(J4-Pin_4): track 0.00 -> 38.5 mm
- net Net-(J4-Pin_3): track 0.00 -> 36.2 mm
- net Net-(J2-Pin_3): track 0.00 -> 34.2 mm
- net Net-(J1-Pin_4): track 0.00 -> 33.1 mm
- net Net-(J3-Pin_3): track 0.00 -> 32.8 mm
- net Net-(J3-Pin_4): track 0.00 -> 31.1 mm
- net Net-(J1-Pin_3): track 0.00 -> 31.0 mm
- net Net-(J2-Pin_4): track 0.00 -> 28.8 mm
- net Net-(U2-EN1,2): track 0.00 -> 28.2 mm
- net Net-(U1-1A): track 0.00 -> 27.2 mm
- net Net-(U1-EN1,2): track 0.00 -> 26.9 mm
- net Net-(U2-1A): track 0.00 -> 26.0 mm
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
Commit message: pcb edit
Routing:
- net GND: track 338.0 -> 356.8 mm
- net Net-(U2-1A): track 26.0 -> 27.4 mm
- net Net-(U2-4A): track 25.5 -> 26.5 mm
- net +5V: track 222.3 -> 223.1 mm
- net Net-(U1-3A): track 14.1 -> 13.4 mm
- net +12V: track 153.9 -> 153.2 mm

Commit message: pcb edit
Routing:
- net GND: track 356.8 -> 355.6 mm
Changed lines of the file:
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@@
+	)
+	(segment
+		(start 116 94.145)
+		(end 118.855 94.145)
+		(width 0.2)
+		(layer "B.Cu")
+		(net 2)
 	)
 	(segment
@@
 	)
 	(segment
-		(start 123.66 92.66)
-		(end 123.66 88.725)
-		(width 0.2)
-		(layer "B.Cu")
-		(net 2)
-	)
-	(segment
 		(start 184.615 76.385)
 		(end 182.92 78.08)
@@
 	)
 	(segment
+		(start 126.145 94.145)
+		(end 123.66 91.66)
+		(width 0.2)
+		(layer "B.Cu")
+		(net 2)
+	)
+	(segment
 		(start 185.145 95.145)
 		(end 182.92 92.92)
@@
 	)
 	(segment
-		(start 116 94.145)
-		(end 119.855 94.145)
+		(start 121.12 91.88)
+		(end 121.12 88.725)
 		(width 0.2)
 		(layer "B.Cu")
@@
 	)
 	(segment
-		(start 119.855 94.145)
-		(end 121.12 92.88)
+		(start 123.66 91.66)
+		(end 123.66 88.725)
 		(width 0.2)
 		(layer "B.Cu")
@@
 	(segment
 		(start 128.5 94.145)
-		(end 125.145 94.145)
+		(end 126.145 94.145)
 		(width 0.2)
 		(layer "B.Cu")
@@
 	)
 	(segment
-		(start 125.145 94.145)
-		(end 123.66 92.66)
-		(width 0.2)
-		(layer "B.Cu")
-		(net 2)
-	)
-	(segment
 		(start 177.855 95.145)
 		(end 180.38 92.62)
@@
 	)
 	(segment
-		(start 121.12 92.88)
-		(end 121.12 88.725)
-		(width 0.2)
-		(layer "B.Cu")
-		(net 2)
-	)
-	(segment
 		(start 119.805 76.805)
 		(end 121.12 78.12)
@@
 		(width 0.2)
 		(layer "B.Cu")
+		(net 2)
+	)
+	(segment
+		(start 118.855 94.145)
+		(end 121.12 91.88)
+		(width 0.2)
+		(layer "B.Cu")

Commit message: direct kinematiks addition
Routing:
- net GND: track 355.6 -> 323.6 mm
- net +12V: track 153.2 -> 153.8 mm

Commit message: pcb edit
Routing:
- net GND: track 323.6 -> 7.24 mm
- net +5V: track 223.4 -> 237.6 mm
- net Net-(J3-Pin_3): track 32.8 -> 28.2 mm
- net Net-(J3-Pin_4): track 31.1 -> 26.7 mm
- net Net-(J1-Pin_4): track 33.1 -> 29.3 mm
- net Net-(J4-Pin_3): track 36.2 -> 32.7 mm
- net Net-(J1-Pin_3): track 31.0 -> 28.2 mm
- net Net-(U2-1A): track 27.4 -> 25.7 mm
- net Net-(J2-Pin_3): track 34.2 -> 32.6 mm
- net Net-(J4-Pin_4): track 38.5 -> 37.0 mm
- net Net-(U2-4A): track 26.5 -> 25.2 mm
- net Net-(U2-EN3,4): track 10.7 -> 9.66 mm
- net Net-(U1-1A): track 27.2 -> 26.4 mm
- net Net-(U2-EN1,2): track 28.2 -> 27.4 mm
- net Net-(U2-2A): track 11.8 -> 11.0 mm
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- added copper zone on B.Cu, net GND

Commit message: pcb correction
Parts:
- moved D5 0.50 mm to (188.0, 66.7)
- moved D6 0.50 mm to (175.5, 66.6)
- moved J3 0.27 mm to (188.0, 62.0)
Routing:
- net Net-(J1-Pin_4): track 29.3 -> 30.8 mm
- net +12V: track 153.8 -> 155.2 mm
- net Net-(U2-4A): track 25.2 -> 26.2 mm
- net +5V: track 237.6 -> 238.4 mm
- net Net-(U2-1A): track 25.7 -> 24.9 mm
- added copper zone on F.Cu, net GND
Other:
- board outline added: 86 x 78.2 mm

Commit message: pcb edit
Routing:
- net +12V: track 155.2 -> 158.0 mm
Changed lines of the file:
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@@
 	)
 	(segment
-		(start 115 124.725)
-		(end 181.4675 124.725)
+		(start 184.5 124.1)
+		(end 184.5 121.6925)
 		(width 0.8)
 		(layer "B.Cu")
@@
 	)
 	(segment
-		(start 110.8 120.525)
-		(end 115 124.725)
-		(width 0.8)
-		(layer "B.Cu")
-		(net 19)
-	)
-	(segment
 		(start 110.8 83.805)
 		(end 110.8 120.525)
@@
 	)
 	(segment
+		(start 182.2 126.4)
+		(end 184.5 124.1)
+		(width 0.8)
+		(layer "B.Cu")
+		(net 19)
+	)
+	(segment
 		(start 191.854774 117.645226)
 		(end 191.854774 90.499774)
@@
 	)
 	(segment
-		(start 181.4675 124.725)
-		(end 184.5 121.6925)
+		(start 116.675 126.4)
+		(end 182.2 126.4)
+		(width 0.8)
+		(layer "B.Cu")
+		(net 19)
+	)
+	(segment
+		(start 110.8 120.525)
+		(end 116.675 126.4)
 		(width 0.8)
 		(layer "B.Cu")
@@
 		(layer "B.Cu")
 		(hatch edge 0.5)
-		(connect_pads
-			(clearance 0.5)
+		(priority 5)
+		(connect_pads
+			(clearance 0.5)
