File: pcb/wheels-pcb/wheels-pcb.kicad_pcb (KiCad board)
At the start: 2 copper layers, 86 x 78.2 mm, 16 parts, among them J1 Motor_1, J2 Motor_2, J3 Motor_3, J4 Motor_4, J5 Conn_01x03, U1 L293D, U2 L293D, U3 ESP32S_38P

Commit message: Micro-Ros code addition (omnidirectional logic)
Routing:
- net GND: track 7.24 -> 10.5 mm
Changed lines of the file:
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@@
+	)
+	(segment
+		(start 178 111.525)
+		(end 178 111.2)
+		(width 0.2)
+		(layer "F.Cu")
+		(net 2)
+	)
+	(segment
+		(start 178 111.2)
+		(end 177 110.2)
+		(width 0.5)
+		(layer "F.Cu")
+		(net 2)
 	)
 	(segment
@@
 		(end 127.8475 76.1525)
 		(width 0.2)
+		(layer "B.Cu")
+		(net 2)
+	)
+	(segment
+		(start 125.875 61.725)
+		(end 124.8 62.8)
+		(width 0.5)
 		(layer "B.Cu")
 		(net 2)
@@
 		(layer "B.Cu")
 		(net 31)
-	)
-	(zone
-		(net 2)
-		(net_name "GND")
-		(layer "F.Cu")
-		(hatch edge 0.5)
-		(priority 1)
-		(connect_pads
-			(clearance 0.5)
-		)
-		(min_thickness 0.25)
-		(filled_areas_thickness no)
-		(fill yes
-			(thermal_gap 0.5)
-			(thermal_bridge_width 0.5)
-		)
-		(polygon
-			(pts
-				(xy 130.4 90) (xy 130.8 90.4) (xy 138.8 90.4) (xy 138.8 88.4) (xy 132.2 88.4) (xy 131.2 89.8) (xy 130.4 89.8)
-			)
-		)
 	)
 	(zone
@@
 			)
 		)
-	)
-	(zone
-		(net 2)
-		(net_name "GND")
-		(layer "F.Cu")
-		(hatch edge 0.5)
-		(priority 4)
-		(connect_pads
-			(clearance 0.5)
-		)
-		(min_thickness 0.25)
-		(filled_areas_thickness no)
-		(fill yes
-			(thermal_gap 0.5)
-			(thermal_bridge_width 0.5)
-		)
-		(polygon
-			(pts
-				(xy 164.6 87.610811) (xy 164.6 93) (xy 168 93) (xy 172.4 88.8) (xy 172.4 87.4)
-			)
-		)
-	)
-	(zone
-		(net 2)
-		(net_name "GND")
-		(layer "F.Cu")
-		(hatch edge 0.5)
-		(priority 2)
-		(connect_pads
-			(clearance 0.5)
-		)
-		(min_thickness 0.25)
-		(filled_areas_thickness no)
-		(fill yes
-			(thermal_gap 0.5)
-			(thermal_bridge_width 0.5)
-		)
-		(polygon
-			(pts
-				(xy 131.4 82.2) (xy 131.4 83) (xy 139.4 83) (xy 139.4 81.4) (xy 132.8 81.4)
-			)
-		)
-	)
-	(zone
-		(net 2)
-		(net_name "GND")
-		(layer "F.Cu")
-		(hatch edge 0.5)
-		(priority 3)
-		(connect_pads
-			(clearance 0.5)
-		)
-		(min_thickness 0.25)
-		(filled_areas_thickness no)
-		(fill yes
-			(thermal_gap 0.5)
-			(thermal_bridge_width 0.5)
-		)
-		(polygon
-			(pts
-				(xy 129.2 89.6) (xy 130.6 91) (xy 139.4 91) (xy 139.4 93.2) (xy 131.4 93.2) (xy 128.2 89.8)
-			)
-		)
