Commit message: gazebo update

File: src/mec_mobile/mec_mobile_description/urdf/robots/robot_omni_3d.urdf.xacro (robot description, xacro)
@@ -1,4 +1,4 @@
 <?xml version="1.0"?>
-<robot xmlns:xacro="http://www.ros.org/wiki/xacro" name="robot_omni_3d">
+<robot xmlns:xacro="http://www.ros.org/wiki/xacro" name="robot_omni_3d" xmlns:gz="http://gazebosim.org/schema">
     <xacro:property name="M_PI" value="3.1415926535897931" />
     <xacro:arg name="robot_name" default="robot_omni_3d"/>
@@ -30,5 +30,5 @@
         side="front_right"
         xyz="-0.11788 -0.081566 -0.037705"
-        rpy="1.5708 0 1.5708"
+        rpy="1.5708 0 -1.5708"
         mesh="fr_wheel_link.STL"/>
     <!-- Rear Right Wheel -->
@@ -37,6 +37,63 @@
         side="back_right"
         xyz="-0.11788 0.081609 -0.037681"
-        rpy="1.5708 0 1.5708"
+        rpy="-1.5708 0 1.5708"
         mesh="rr_wheel_link.STL"/>
+ <gazebo reference='front_left_wheel_link'>
+    <collision>
+      <surface>
+        <friction>
+          <ode>
+            <mu>1.5</mu>
+            <mu2>0.0</mu2>
+            <fdir1 gz:expressed_in="base_footprint">1 -1 0</fdir1>
+          </ode>
+        </friction>
+      </surface>
+    </collision>
+  </gazebo>
+  <gazebo reference='back_left_wheel_link'>
+    <collision>
+      <surface>
+        <friction>
+          <ode>
+            <mu>1.5</mu>
+            <mu2>0.0</mu2>
+            <fdir1 gz:expressed_in="base_footprint">1 1 0</fdir1>
+          </ode>
+        </friction>
+      </surface>
+    </collision>
+  </gazebo>
+  <gazebo reference='front_right_wheel_link'>
+    <collision>
+      <surface>
+        <friction>
+          <ode>
+            <mu>1.5</mu>
+            <mu2>0.0</mu2>
+            <fdir1 gz:expressed_in="base_footprint">1 1 0</fdir1>
+          </ode>
+        </friction>
+      </surface>
+    </collision>
+  </gazebo>
+  <gazebo reference='back_right_wheel_link'>
+    <collision>
+      <surface>
+        <friction>
+          <ode>
+            <mu>1.5</mu>
+            <mu2>0.0</mu2>
+            <fdir1 gz:expressed_in="base_footprint">1 -1 0</fdir1>
+          </ode>
+        </friction>
+      </surface>
+    </collision>
+  </gazebo>
+  <gazebo reference="base_link">
+    <mu1>0.000002</mu1>
+    <mu2>0.000002</mu2>
+    <!-- <material>Gazebo/Red</material> -->
+  </gazebo>
     <!-- Arm -->
     <xacro:arm prefix="$(arg prefix)"/>
